File: game-on.kicad_sch (KiCad schematic)
At the start: 9 parts, among them X1 #badgelife

Commit message: Tweaked a few values
Connections:
- no-connect marks 11 -> 7
Other:
- sheet RP2040 ports: added none; removed RX1, SWDCLK, SWDIO, TX1
Changed lines of the file:
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@@
   (no_connect (at 161.29 99.06))
   (no_connect (at 161.29 86.36))
-  (no_connect (at 161.29 73.66))
-  (no_connect (at 116.84 78.74))
-  (no_connect (at 116.84 81.28))
   (no_connect (at 116.84 93.98))
-  (no_connect (at 161.29 76.2))
   (no_connect (at 161.29 78.74))
   (no_connect (at 161.29 81.28))
@@
       (effects (font (size 1.27 1.27)) (justify left top))
     )
-    (pin "SWDCLK" input (at 116.84 78.74 180)
-      (effects (font (size 1.27 1.27)) (justify left))
-    )
-    (pin "SWDIO" input (at 116.84 81.28 180)
-      (effects (font (size 1.27 1.27)) (justify left))
-    )
     (pin "RTS1{slash}AUD_BCLK" input (at 161.29 78.74 0)
-      (effects (font (size 1.27 1.27)) (justify right))
-    )
-    (pin "TX1" input (at 161.29 73.66 0)
-      (effects (font (size 1.27 1.27)) (justify right))
-    )
-    (pin "RX1" input (at 161.29 76.2 0)
       (effects (font (size 1.27 1.27)) (justify right))
     )
@@
     )
     (path "/66a007aa-690f-49cd-ac96-98fe74602400/5ad664c3-f356-4841-8269-82adc30d86c0"
-      (reference "C15") (unit 1) (value "15pF") (footprint "Capacitor_SMD:C_0603_1608Metric")
+      (reference "C15") (unit 1) (value "30pF") (footprint "Capacitor_SMD:C_0603_1608Metric")
     )
     (path "/66a007aa-690f-49cd-ac96-98fe74602400/ea91146b-c19d-4537-8775-9f2d267eaaf0"
-      (reference "C16") (unit 1) (value "15pF") (footprint "Capacitor_SMD:C_0603_1608Metric")
+      (reference "C16") (unit 1) (value "30pF") (footprint "Capacitor_SMD:C_0603_1608Metric")
     )
     (path "/66a007aa-690f-49cd-ac96-98fe74602400/c9ca9cc8-0d9a-4009-b2ce-622ed1a311be"
@@
     )
     (path "/c02f64c6-7bbb-4eb3-b45b-4884d1936fa5/e6397214-9de1-40c7-a9f2-7d9fe1229f81"
-      (reference "R6") (unit 1) (value "22R") (footprint "Resistor_SMD:R_0603_1608Metric")
+      (reference "R6") (unit 1) (value "27R") (footprint "Resistor_SMD:R_0603_1608Metric")
     )
     (path "/66a007aa-690f-49cd-ac96-98fe74602400/fd512a0a-8aa8-4c8b-a8c7-87b1941096a0"
@@
     )
     (path "/66a007aa-690f-49cd-ac96-98fe74602400/310fe9e5-1690-4a7e-bc0e-07816d458a90"
-      (reference "R13") (unit 1) (value "27") (footprint "Resistor_SMD:R_0603_1608Metric")
+      (reference "R13") (unit 1) (value "27R") (footprint "Resistor_SMD:R_0603_1608Metric")
     )
     (path "/66a007aa-690f-49cd-ac96-98fe74602400/d0e4cb32-8594-4bd2-9097-a3cd4b6c61a5"
-      (reference "R14") (unit 1) (value "27") (footprint "Resistor_SMD:R_0603_1608Metric")
+      (reference "R14") (unit 1) (value "27R") (footprint "Resistor_SMD:R_0603_1608Metric")
     )
     (path "/877ac62c-7fa2-4c18-8d3c-0d6e89de9449/533ac147-192e-43e4-b55c-d5c862a6a445"
