File: rp2040.kicad_sch (KiCad schematic)
At the start: 31 parts, among them J1 USB_C, J2 Qwiic, J3 DEBUG, SW6 RESET, SW7 BOOT, U4 W25QXX128MBIT, U5 RP2040, Y1 12MHz

Commit message: Tweaked a few values
Parts:
- C15, C16: value 15pF -> 30pF
- R13, R14: value 27 -> 27R
Changed lines of the file:
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@@
     (in_bom yes) (on_board yes)
     (property "Reference" "R13" (id 0) (at 196.85 73.66 90))
-    (property "Value" "27" (id 1) (at 196.85 76.2 90))
+    (property "Value" "27R" (id 1) (at 196.85 76.2 90))
     (property "Footprint" "Resistor_SMD:R_0603_1608Metric" (id 2) (at 196.85 77.978 90)
       (effects (font (size 1.27 1.27)) hide)
@@
     (in_bom yes) (on_board yes)
     (property "Reference" "C15" (id 0) (at 187.96 85.09 90))
-    (property "Value" "15pF" (id 1) (at 187.96 87.63 90))
+    (property "Value" "30pF" (id 1) (at 187.96 87.63 90))
     (property "Footprint" "Capacitor_SMD:C_0603_1608Metric" (id 2) (at 191.77 90.4748 0)
       (effects (font (size 1.27 1.27)) hide)
@@
     (in_bom yes) (on_board yes)
     (property "Reference" "R14" (id 0) (at 196.85 81.28 90))
-    (property "Value" "27" (id 1) (at 196.85 78.74 90))
+    (property "Value" "27R" (id 1) (at 196.85 78.74 90))
     (property "Footprint" "Resistor_SMD:R_0603_1608Metric" (id 2) (at 196.85 80.518 90)
       (effects (font (size 1.27 1.27)) hide)
@@
     (in_bom yes) (on_board yes)
     (property "Reference" "C16" (id 0) (at 187.96 105.41 90))
-    (property "Value" "15pF" (id 1) (at 187.96 102.87 90))
+    (property "Value" "30pF" (id 1) (at 187.96 102.87 90))
     (property "Footprint" "Capacitor_SMD:C_0603_1608Metric" (id 2) (at 191.77 98.0948 0)
       (effects (font (size 1.27 1.27)) hide)
