File: st7735S_spi_display.kicad_sch (KiCad schematic)
At the start: 4 parts, among them Q3 BC817, U3 ST7735S-SPI-14pin

Commit message: Tweaked a few values
Parts:
- R6: value 22R -> 27R
Changed lines of the file:
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@@
     (in_bom yes) (on_board yes) (fields_autoplaced)
     (property "Reference" "R6" (id 0) (at 101.6 83.82 90))
-    (property "Value" "22R" (id 1) (at 101.6 86.36 90))
+    (property "Value" "27R" (id 1) (at 101.6 86.36 90))
     (property "Footprint" "Resistor_SMD:R_0603_1608Metric" (id 2) (at 101.6 87.122 90)
       (effects (font (size 1.27 1.27)) hide)
